File: Hardware/lcd_board/lcd_board.sch (KiCad schematic (older format))
At the start: 13 parts, among them J1 Conn_01x40, J2 Conn_01x16, U1 74HC04, U2 74HC173, U3 74HC173, U4 74HC174

Commit message: LCD board with through hole components
Parts:
- C1, C2, C3, C4, C5: value C_Small -> 4.7u; footprint Capacitor_SMD:C_1206_3216Metric_Pad1.42x1.75mm_HandSolder -> Capacitor_THT:C_Disc_D4.3mm_W1.9mm_P5.00mm
- R1: footprint Resistor_SMD:R_0805_2012Metric_Pad1.15x1.40mm_HandSolder -> Resistor_THT:R_Axial_DIN0204_L3.6mm_D1.6mm_P5.08mm_Horizontal
- U4: value 74HC174 -> 74HC173
Changed lines of the file:
@@
 P 7650 5300
 F 0 "U4" H 7650 6381 50  0000 C CNN
-F 1 "74HC174" H 7650 6290 50  0000 C CNN
+F 1 "74HC173" H 7650 6290 50  0000 C CNN
 F 2 "Package_DIP:DIP-16_W7.62mm_Socket" H 7650 5300 50  0001 C CNN
 F 3 "http://www.ti.com/lit/gpn/sn74LS04" H 7650 5300 50  0001 C CNN
@@
 P 7900 4150
 F 0 "C4" V 7671 4150 50  0000 C CNN
-F 1 "C_Small" V 7762 4150 50  0000 C CNN
-F 2 "Capacitor_SMD:C_1206_3216Metric_Pad1.42x1.75mm_HandSolder" H 7900 4150 50  0001 C CNN
+F 1 "4.7u" V 7762 4150 50  0000 C CNN
+F 2 "Capacitor_THT:C_Disc_D4.3mm_W1.9mm_P5.00mm" H 7900 4150 50  0001 C CNN
 F 3 "~" H 7900 4150 50  0001 C CNN
 	1    7900 4150
@@
 P 6350 3750
 F 0 "C3" V 6121 3750 50  0000 C CNN
-F 1 "C_Small" V 6212 3750 50  0000 C CNN
-F 2 "Capacitor_SMD:C_1206_3216Metric_Pad1.42x1.75mm_HandSolder" H 6350 3750 50  0001 C CNN
+F 1 "4.7u" V 6212 3750 50  0000 C CNN
+F 2 "Capacitor_THT:C_Disc_D4.3mm_W1.9mm_P5.00mm" H 6350 3750 50  0001 C CNN
 F 3 "~" H 6350 3750 50  0001 C CNN
 	1    6350 3750
@@
 P 6350 850
 F 0 "C2" V 6121 850 50  0000 C CNN
-F 1 "C_Small" V 6212 850 50  0000 C CNN
-F 2 "Capacitor_SMD:C_1206_3216Metric_Pad1.42x1.75mm_HandSolder" H 6350 850 50  0001 C CNN
+F 1 "4.7u" V 6212 850 50  0000 C CNN
+F 2 "Capacitor_THT:C_Disc_D4.3mm_W1.9mm_P5.00mm" H 6350 850 50  0001 C CNN
 F 3 "~" H 6350 850 50  0001 C CNN
 	1    6350 850
@@
 P 4750 5250
 F 0 "C1" V 4521 5250 50  0000 C CNN
-F 1 "C_Small" V 4612 5250 50  0000 C CNN
-F 2 "Capacitor_SMD:C_1206_3216Metric_Pad1.42x1.75mm_HandSolder" H 4750 5250 50  0001 C CNN
+F 1 "4.7u" V 4612 5250 50  0000 C CNN
+F 2 "Capacitor_THT:C_Disc_D4.3mm_W1.9mm_P5.00mm" H 4750 5250 50  0001 C CNN
 F 3 "~" H 4750 5250 50  0001 C CNN
 	1    4750 5250
@@
 F 0 "R1" V 8604 4700 50  0000 C CNN
 F 1 "330R" V 8695 4700 50  0000 C CNN
-F 2 "Resistor_SMD:R_0805_2012Metric_Pad1.15x1.40mm_HandSolder" H 8800 4700 50  0001 C CNN
+F 2 "Resistor_THT:R_Axial_DIN0204_L3.6mm_D1.6mm_P5.08mm_Horizontal" H 8800 4700 50  0001 C CNN
 F 3 "~" H 8800 4700 50  0001 C CNN
 	1    8800 4700
@@
 P 8400 2150
 F 0 "C5" V 8171 2150 50  0000 C CNN
-F 1 "C_Small" V 8262 2150 50  0000 C CNN
-F 2 "Capacitor_SMD:C_1206_3216Metric_Pad1.42x1.75mm_HandSolder" H 8400 2150 50  0001 C CNN
+F 1 "4.7u" V 8262 2150 50  0000 C CNN
+F 2 "Capacitor_THT:C_Disc_D4.3mm_W1.9mm_P5.00mm" H 8400 2150 50  0001 C CNN
 F 3 "~" H 8400 2150 50  0001 C CNN
 	1    8400 2150

Commit message: final update for through hole conversion
Parts:
- C1, C2, C3, C4, C5: value 4.7u -> 10n
Changed lines of the file:
@@
 P 7900 4150
 F 0 "C4" V 7671 4150 50  0000 C CNN
-F 1 "4.7u" V 7762 4150 50  0000 C CNN
+F 1 "10n" V 7762 4150 50  0000 C CNN
 F 2 "Capacitor_THT:C_Disc_D4.3mm_W1.9mm_P5.00mm" H 7900 4150 50  0001 C CNN
 F 3 "~" H 7900 4150 50  0001 C CNN
@@
 P 6350 3750
 F 0 "C3" V 6121 3750 50  0000 C CNN
-F 1 "4.7u" V 6212 3750 50  0000 C CNN
+F 1 "10n" V 6212 3750 50  0000 C CNN
 F 2 "Capacitor_THT:C_Disc_D4.3mm_W1.9mm_P5.00mm" H 6350 3750 50  0001 C CNN
 F 3 "~" H 6350 3750 50  0001 C CNN
@@
 P 6350 850
 F 0 "C2" V 6121 850 50  0000 C CNN
-F 1 "4.7u" V 6212 850 50  0000 C CNN
+F 1 "10n" V 6212 850 50  0000 C CNN
 F 2 "Capacitor_THT:C_Disc_D4.3mm_W1.9mm_P5.00mm" H 6350 850 50  0001 C CNN
 F 3 "~" H 6350 850 50  0001 C CNN
@@
 P 4750 5250
 F 0 "C1" V 4521 5250 50  0000 C CNN
-F 1 "4.7u" V 4612 5250 50  0000 C CNN
+F 1 "10n" V 4612 5250 50  0000 C CNN
 F 2 "Capacitor_THT:C_Disc_D4.3mm_W1.9mm_P5.00mm" H 4750 5250 50  0001 C CNN
 F 3 "~" H 4750 5250 50  0001 C CNN
@@
 P 8400 2150
 F 0 "C5" V 8171 2150 50  0000 C CNN
-F 1 "4.7u" V 8262 2150 50  0000 C CNN
+F 1 "10n" V 8262 2150 50  0000 C CNN
 F 2 "Capacitor_THT:C_Disc_D4.3mm_W1.9mm_P5.00mm" H 8400 2150 50  0001 C CNN
 F 3 "~" H 8400 2150 50  0001 C CNN

Commit message: update lcd board with bigger resistors
Parts:
- R1: footprint Resistor_THT:R_Axial_DIN0204_L3.6mm_D1.6mm_P5.08mm_Horizontal -> Resistor_THT:R_Axial_DIN0207_L6.3mm_D2.5mm_P10.16mm_Horizontal
Other:
- note removed: "TODO check the order of the two pins"
Changed lines of the file:
@@
 	1    0    0    -1
 $EndComp
-Text Notes 10350 4250 2    50   ~ 0
-TODO check the order of the two pins
 $Comp
 L Device:R_Small R1
@@
 F 0 "R1" V 8604 4700 50  0000 C CNN
 F 1 "330R" V 8695 4700 50  0000 C CNN
-F 2 "Resistor_THT:R_Axial_DIN0204_L3.6mm_D1.6mm_P5.08mm_Horizontal" H 8800 4700 50  0001 C CNN
+F 2 "Resistor_THT:R_Axial_DIN0207_L6.3mm_D2.5mm_P10.16mm_Horizontal" H 8800 4700 50  0001 C CNN
 F 3 "~" H 8800 4700 50  0001 C CNN
 	1    8800 4700
