File: Hardware/lcd_board/lcd_board.kicad_pcb (KiCad board)
At the start: 2 copper layers, 80.8 x 60.1 mm, 18 parts, among them J1 Conn_01x40, J2 Conn_01x16, U1 74HC04, U2 74HC173, U3 74HC173, U4 74HC173

Commit message: Add job for LCD board + update to kicad 6
Parts:
- RV1: value R_POT_Small -> 10k
- moved C1 173.9 mm to (122.3, 132.5)
- moved C5 173.9 mm to (100.2, 97.0)
- moved J1 173.9 mm to (175.9, 137.3)
- moved J2 173.9 mm to (139.1, 94.0)
- moved U2 173.9 mm to (173.4, 105.5)
- moved C2 173.9 mm to (126.6, 108.1)
- moved C3 173.9 mm to (168.3, 116.2)
- moved C4 173.9 mm to (152.5, 108.3)
- moved G*** 173.9 mm to (154.8, 88.0) (x2)
- moved R1 173.9 mm to (146.9, 97.7)
- moved REF** 173.9 mm to (173.4, 98.4)
- moved REF** 173.9 mm to (167.3, 98.4)
- moved REF** 173.9 mm to (106.3, 133.0)
- moved RV1 173.9 mm to (174.6, 91.4)
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Connections:
- net R~W~ renamed R~{W}
- net ~INH~ renamed ~{INH}
- net ~IRQ~ renamed ~{IRQ}
- net ~NMI~ renamed ~{NMI}
- net ~RESET~ renamed ~{RESET}
- net ~SLOT_IRQ~ renamed ~{SLOT_IRQ}
- net ~SLOT_SEL~ renamed ~{SLOT_SEL}
- net ~SLOW~ renamed ~{SLOW}
- net ~SSEL~ renamed ~{SSEL}
- U1 pad 10: Net-(U1-Pad10) -> unconnected-(U1-Pad10)
- U1 pad 12: Net-(U1-Pad12) -> unconnected-(U1-Pad12)
- U1 pad 4: Net-(U1-Pad4) -> unconnected-(U1-Pad4)
- U1 pad 6: Net-(U1-Pad6) -> unconnected-(U1-Pad6)
- U1 pad 8: Net-(U1-Pad8) -> unconnected-(U1-Pad8)
- U2 pad 11: Net-(U2-Pad11) -> GND
- U2 pad 12: Net-(U2-Pad12) -> GND
- U2 pad 5: Net-(U2-Pad5) -> unconnected-(U2-Pad5)
- U2 pad 6: Net-(U2-Pad6) -> unconnected-(U2-Pad6)
Routing:
- net GND: track 1.01 -> 0.00 mm
Other:
- net class Default removed
- board text added: "LCD BOARD ${VERSION}"
- board text removed: "LCD BOARD V1.0"
