File: Hardware/lcd_board/lcd_board.kicad_pcb (KiCad board)
At the start: 2 copper layers, 80.8 x 60.1 mm, 18 parts, among them J1 Conn_01x40, J2 Conn_01x16, U1 74HC04, U2 74HC173, U3 74HC173, U4 74HC173

Commit message: Add R/W to LCD board enable
Connections:
- U2 pad 10: ~{SLOT_SEL} -> R~{W}
- U3 pad 10: ~{SLOT_SEL} -> R~{W}
- U4 pad 10: ~{SLOT_SEL} -> R~{W}
Routing:
- net R~{W}: track 0.00 -> 92.5 mm, vias 0 -> 3
Changed lines of the file:
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@@
       (net 45 "~{SLOT_SEL}") (pinfunction "E1") (pintype "input"))
     (pad "10" thru_hole oval (at 7.62 15.24 270) (size 1.6 1.6) (drill 0.8) (layers *.Cu *.Mask)
-      (net 45 "~{SLOT_SEL}") (pinfunction "E2") (pintype "input"))
+      (net 39 "R~{W}") (pinfunction "E2") (pintype "input"))
     (pad "11" thru_hole oval (at 7.62 12.7 270) (size 1.6 1.6) (drill 0.8) (layers *.Cu *.Mask)
       (net 7 "GND") (pinfunction "D3") (pintype "input"))
@@
       (net 45 "~{SLOT_SEL}") (pinfunction "E1") (pintype "input"))
     (pad "10" thru_hole oval (at 7.62 15.24 270) (size 1.6 1.6) (drill 0.8) (layers *.Cu *.Mask)
-      (net 45 "~{SLOT_SEL}") (pinfunction "E2") (pintype "input"))
+      (net 39 "R~{W}") (pinfunction "E2") (pintype "input"))
     (pad "11" thru_hole oval (at 7.62 12.7 270) (size 1.6 1.6) (drill 0.8) (layers *.Cu *.Mask)
       (net 20 "D3") (pinfunction "D3") (pintype "input"))
@@
       (net 45 "~{SLOT_SEL}") (pinfunction "E1") (pintype "input"))
     (pad "10" thru_hole oval (at 7.62 15.24 270) (size 1.6 1.6) (drill 0.8) (layers *.Cu *.Mask)
-      (net 45 "~{SLOT_SEL}") (pinfunction "E2") (pintype "input"))
+      (net 39 "R~{W}") (pinfunction "E2") (pintype "input"))
     (pad "11" thru_hole oval (at 7.62 12.7 270) (size 1.6 1.6) (drill 0.8) (layers *.Cu *.Mask)
       (net 12 "D7") (pinfunction "D3") (pintype "input"))
@@
   (segment (start 126.619 113.077) (end 126.191 112.649) (width 1) (layer "F.Cu") (net 8))
   (segment (start 147.955 139.827) (end 145.415 137.287) (width 1) (layer "F.Cu") (net 8))
-  (via (at 123.571 110.109) (size 0.8) (drill 0.4) (layers "F.Cu" "B.Cu") (net 8))
-  (segment (start 123.571 112.649) (end 123.571 110.109) (width 1) (layer "B.Cu") (net 8))
+  (via (at 123.500994 109.8925) (size 0.8) (drill 0.4) (layers "F.Cu" "B.Cu") (net 8))
+  (segment (start 123.571 109.962506) (end 123.500994 109.8925) (width 1) (layer "B.Cu") (net 8))
+  (segment (start 123.571 112.649) (end 123.571 109.962506) (width 1) (layer "B.Cu") (net 8))
   (segment (start 154.780999 138.651999) (end 154.210001 138.081001) (width 0.25) (layer "F.Cu") (net 12))
   (segment (start 158.115 139.827) (end 156.939999 138.651999) (width 0.25) (layer "F.Cu") (net 12))
@@
   (segment (start 126.002999 123.107501) (end 127.254 121.8565) (width 0.5) (layer "B.Cu") (net 28))
   (segment (start 126.002999 125.457001) (end 126.002999 123.107501) (width 0.5) (layer "B.Cu") (net 28))
-  (segment (start 131.699 113.03) (end 134.239 113.03) (width 0.5) (layer "F.Cu") (net 45))
-  (segment (start 129.9845 111.3155) (end 131.699 113.03) (width 0.5) (layer "F.Cu") (net 45))
-  (segment (start 154.261499 111.779999) (end 155.6385 113.157) (width 0.5) (layer "F.Cu") (net 45))
-  (segment (start 109.6645 111.3155) (end 129.9845 111.3155) (width 0.5) (layer "F.Cu") (net 45))
-  (segment (start 136.525 127.8255) (end 136.525 132.334002) (width 0.5) (layer "F.Cu") (net 45))
-  (segment (start 134.239 113.03) (end 135.489001 111.779999) (width 0.5) (layer "F.Cu") (net 45))
-  (segment (start 135.489001 111.779999) (end 154.261499 111.779999) (width 0.5) (layer "F.Cu") (net 45))
-  (segment (start 125.4125 116.713) (end 136.525 127.8255) (width 0.5) (layer "F.Cu") (net 45))
-  (segment (start 112.395 116.713) (end 125.4125 116.713) (width 0.5) (layer "F.Cu") (net 45))
-  (segment (start 155.6385 113.157) (end 158.1785 113.157) (width 0.5) (layer "F.Cu") (net 45))
-  (segment (start 105.791 112.649) (end 108.331 112.649) (width 0.5) (layer "F.Cu") (net 45))
-  (segment (start 108.331 112.649) (end 109.6645 111.3155) (width 0.5) (layer "F.Cu") (net 45))
-  (segment (start 108.331 112.649) (end 112.395 116.713) (width 0.5) (layer "F.Cu") (net 45))
+  (segment (start 132.283499 111.074499) (end 109.905501 111.074499) (width 0.25) (layer "F.Cu") (net 39))
+  (segment (start 123.589 136.253) (end 123.589 124.819978) (width 0.25) (layer "F.Cu") (net 39))
+  (segment (start 156.476999 111.455499) (end 158.1785 113.157) (width 0.25) (layer "F.Cu") (net 39))
+  (segment (start 122.555 137.287) (end 123.589 136.253) (width 0.25) (layer "F.Cu") (net 39))
+  (segment (start 134.239 113.03) (end 135.813501 111.455499) (width 0.25) (layer "F.Cu") (net 39))
+  (segment (start 126.014 120.807) (end 125.73 120.523) (width 0.25) (layer "F.Cu") (net 39))
+  (segment (start 135.813501 111.455499) (end 156.476999 111.455499) (width 0.25) (layer "F.Cu") (net 39))
+  (segment (start 134.239 113.03) (end 132.283499 111.074499) (width 0.25) (layer "F.Cu") (net 39))
+  (segment (start 109.905501 111.074499) (end 108.331 112.649) (width 0.25) (layer "F.Cu") (net 39))
+  (segment (start 123.589 124.819978) (end 126.014 122.394978) (width 0.25) (layer "F.Cu") (net 39))
+  (segment (start 114.3 118.999) (end 109.474 114.173) (width 0.25) (layer "F.Cu") (net 39))
+  (segment (start 125.349 118.999) (end 114.3 118.999) (width 0.25) (layer "F.Cu") (net 39))
+  (segment (start 126.014 122.394978) (end 126.014 120.807) (width 0.25) (layer "F.Cu") (net 39))
+  (via (at 109.474 114.173) (size 0.6) (drill 0.3) (layers "F.Cu" "B.Cu") (net 39))
+  (via (at 125.349 118.999) (size 0.6) (drill 0.3) (layers "F.Cu" "B.Cu") (net 39))
+  (via (at 125.73 120.523) (size 0.6) (drill 0.3) (layers "F.Cu" "B.Cu") (net 39))
+  (segment (start 125.349 120.142) (end 125.349 118.999) (width 0.25) (layer "B.Cu") (net 39))
+  (segment (start 109.474 114.173) (end 109.474 113.792) (width 0.25) (layer "B.Cu") (net 39))
+  (segment (start 125.73 120.523) (end 125.349 120.142) (width 0.25) (layer "B.Cu") (net 39))
+  (segment (start 109.474 113.792) (end 108.331 112.649) (width 0.25) (layer "B.Cu") (net 39))
+  (segment (start 113.0405 119.8985) (end 127.546 119.8985) (width 0.25) (layer "F.Cu") (net 45))
+  (segment (start 136.313009 111.905) (end 135.382 112.836009) (width 0.25) (layer "F.Cu") (net 45))
+  (segment (start 105.791 112.649) (end 106.8705 113.7285) (width 0.25) (layer "F.Cu") (net 45))
+  (segment (start 131.699 113.03) (end 130.193 111.524) (width 0.25) (layer "F.Cu") (net 45))
+  (segment (start 127.546 119.8985) (end 136.525 128.8775) (width 0.25) (layer "F.Cu") (net 45))
+  (segment (start 130.193 111.524) (end 110.405009 111.524) (width 0.25) (layer "F.Cu") (net 45))
+  (segment (start 109.746 112.824991) (end 108.796991 113.774) (width 0.25) (layer "F.Cu") (net 45))
+  (segment (start 109.746 112.183009) (end 109.746 112.824991) (width 0.25) (layer "F.Cu") (net 45))
+  (segment (start 136.525 128.8775) (end 136.525 132.334002) (width 0.25) (layer "F.Cu") (net 45))
+  (segment (start 106.8705 113.7285) (end 113.0405 119.8985) (width 0.25) (layer "F.Cu") (net 45))
+  (segment (start 155.6385 113.157) (end 154.3865 111.905) (width 0.25) (layer "F.Cu") (net 45))
+  (segment (start 110.405009 111.524) (end 109.746 112.183009) (width 0.25) (layer "F.Cu") (net 45))
+  (segment (start 154.3865 111.905) (end 136.313009 111.905) (width 0.25) (layer "F.Cu") (net 45))
+  (segment (start 106.916 113.774) (end 106.8705 113.7285) (width 0.25) (layer "F.Cu") (net 45))
+  (segment (start 132.824 114.155) (end 131.699 113.03) (width 0.25) (layer "F.Cu") (net 45))
+  (segment (start 135.382 112.836009) (end 135.382 113.477991) (width 0.25) (layer "F.Cu") (net 45))
+  (segment (start 134.704991 114.155) (end 132.824 114.155) (width 0.25) (layer "F.Cu") (net 45))
+  (segment (start 135.382 113.477991) (end 134.704991 114.155) (width 0.25) (layer "F.Cu") (net 45))
+  (segment (start 108.796991 113.774) (end 106.916 113.774) (width 0.25) (layer "F.Cu") (net 45))
   (via (at 136.525 132.334002) (size 0.6) (drill 0.3) (layers "F.Cu" "B.Cu") (net 45))
   (segment (start 137.795 139.827) (end 136.525 138.557) (width 0.25) (layer "B.Cu") (net 45))
