File: Hardware/proc_board/proc_board.sch (KiCad schematic (older format))
At the start: 11 parts, among them J1 Conn_01x40, U1 GAL16V8, U2 W65C02SxP, U3 HM62256BLP, U4 28C256

Commit message: Backplane provides diode and pullups for SLOW signal
Parts:
- removed D1: 1N4148, Diode_THT:D_DO-35_SOD27_P7.62mm_Horizontal, symbol pspice:DIODE
- removed R1: 4.7k, Resistor_SMD:R_0805_2012Metric_Pad1.15x1.40mm_HandSolder, symbol Device:R_Small
Connections:
- wire segments 50 -> 47
Other:
- note added: "Diode + pullup provided by backplane"
- note removed: "Added diode + pullup here"
Changed lines of the file:
@@
 Text GLabel 3150 6200 2    50   Output ~ 0
 ~ROM_CS~
-Text GLabel 4500 6350 2    50   Output ~ 0
+Text GLabel 3150 6350 2    50   Output ~ 0
 ~SLOW~
 Wire Wire Line
@@
 Text Notes 1200 7000 0    50   ~ 0
 Added RW here
-Text Notes 3150 6750 0    50   ~ 0
-Added diode + pullup here
-$Comp
-L pspice:DIODE D1
-U 1 1 60359E86
-P 4050 6350
-F 0 "D1" H 4050 6615 50  0000 C CNN
-F 1 "1N4148" H 4050 6524 50  0000 C CNN
-F 2 "Diode_THT:D_DO-35_SOD27_P7.62mm_Horizontal" H 4050 6350 50  0001 C CNN
-F 3 "~" H 4050 6350 50  0001 C CNN
-	1    4050 6350
-	-1   0    0    1
-$EndComp
+Text Notes 3100 6550 0    50   ~ 0
+Diode + pullup provided by backplane
 Wire Wire Line
-	4500 6350 4350 6350
-Wire Wire Line
-	3100 6350 3850 6350
-$Comp
-L Device:R_Small R1
-U 1 1 6035C6C6
-P 4350 6050
-F 0 "R1" H 4409 6096 50  0000 L CNN
-F 1 "4.7k" H 4409 6005 50  0000 L CNN
-F 2 "Resistor_SMD:R_0805_2012Metric_Pad1.15x1.40mm_HandSolder" H 4350 6050 50  0001 C CNN
-F 3 "~" H 4350 6050 50  0001 C CNN
-	1    4350 6050
-	1    0    0    -1
-$EndComp
-$Comp
-L power:+5V #PWR0113
-U 1 1 6035CE86
-P 4350 5950
-F 0 "#PWR0113" H 4350 5800 50  0001 C CNN
-F 1 "+5V" H 4365 6123 50  0000 C CNN
-F 2 "" H 4350 5950 50  0001 C CNN
-F 3 "" H 4350 5950 50  0001 C CNN
-	1    4350 5950
-	1    0    0    -1
-$EndComp
-Wire Wire Line
-	4350 6150 4350 6350
-Connection ~ 4350 6350
-Wire Wire Line
-	4350 6350 4250 6350
+	3150 6350 3100 6350
 $EndSCHEMATC

Commit message: Through hole components for processor board
Parts:
- added J2: Conn_01x14, Connector_PinSocket_2.54mm:PinSocket_1x14_P2.54mm_Vertical, symbol Connector_Generic:Conn_01x14
- C1, C2, C3, C4: value C_Small -> 4.7u; footprint Capacitor_SMD:C_1206_3216Metric_Pad1.42x1.75mm_HandSolder -> Capacitor_THT:C_Disc_D4.3mm_W1.9mm_P5.00mm
- U4: footprint Socket:DIP_Socket-28_W11.9_W12.7_W15.24_W17.78_W18.5_3M_228-1277-00-0602J -> Package_DIP:DIP-28_W15.24mm_Socket
Connections:
- net +5V: now also J2.1 (Pin_1)
- net A10: now also J2.8 (Pin_8)
- net A11: now also J2.6 (Pin_6)
- net A13: now also J2.3 (Pin_3)
- net A8: now also J2.4 (Pin_4)
- net A9: now also J2.5 (Pin_5)
- net D3: now also J2.14 (Pin_14)
- net D4: now also J2.13 (Pin_13)
- net D5: now also J2.12 (Pin_12)
- net D6: now also J2.11 (Pin_11)
- net D7: now also J2.10 (Pin_10)
- net GND: now also J2.7 (Pin_7)
- net ~RAMW~: now also J2.2 (Pin_2)
- net ~RAM_CS~: now also J2.9 (Pin_9)
Other:
- note removed: "Added RW here"
Changed lines of the file:
@@
 P 4800 1700
 F 0 "C3" V 4571 1700 50  0000 C CNN
-F 1 "C_Small" V 4662 1700 50  0000 C CNN
-F 2 "Capacitor_SMD:C_1206_3216Metric_Pad1.42x1.75mm_HandSolder" H 4800 1700 50  0001 C CNN
+F 1 "4.7u" V 4662 1700 50  0000 C CNN
+F 2 "Capacitor_THT:C_Disc_D4.3mm_W1.9mm_P5.00mm" H 4800 1700 50  0001 C CNN
 F 3 "~" H 4800 1700 50  0001 C CNN
 	1    4800 1700
@@
 F 0 "U4" H 9500 4731 50  0000 C CNN
 F 1 "28C256" H 9500 4640 50  0000 C CNN
-F 2 "Socket:DIP_Socket-28_W11.9_W12.7_W15.24_W17.78_W18.5_3M_228-1277-00-0602J" H 9500 3450 50  0001 C CNN
+F 2 "Package_DIP:DIP-28_W15.24mm_Socket" H 9500 3450 50  0001 C CNN
 F 3 "http://ww1.microchip.com/downloads/en/DeviceDoc/doc0006.pdf" H 9500 3450 50  0001 C CNN
 	1    9500 3450
@@
 P 7800 2300
 F 0 "C1" V 7571 2300 50  0000 C CNN
-F 1 "C_Small" V 7662 2300 50  0000 C CNN
-F 2 "Capacitor_SMD:C_1206_3216Metric_Pad1.42x1.75mm_HandSolder" H 7800 2300 50  0001 C CNN
+F 1 "4.7u" V 7662 2300 50  0000 C CNN
+F 2 "Capacitor_THT:C_Disc_D4.3mm_W1.9mm_P5.00mm" H 7800 2300 50  0001 C CNN
 F 3 "~" H 7800 2300 50  0001 C CNN
 	1    7800 2300
@@
 P 9700 2100
 F 0 "C2" V 9471 2100 50  0000 C CNN
-F 1 "C_Small" V 9562 2100 50  0000 C CNN
-F 2 "Capacitor_SMD:C_1206_3216Metric_Pad1.42x1.75mm_HandSolder" H 9700 2100 50  0001 C CNN
+F 1 "4.7u" V 9562 2100 50  0000 C CNN
+F 2 "Capacitor_THT:C_Disc_D4.3mm_W1.9mm_P5.00mm" H 9700 2100 50  0001 C CNN
 F 3 "~" H 9700 2100 50  0001 C CNN
 	1    9700 2100
@@
 P 2450 5500
 F 0 "C4" V 2221 5500 50  0000 C CNN
-F 1 "C_Small" V 2312 5500 50  0000 C CNN
-F 2 "Capacitor_SMD:C_1206_3216Metric_Pad1.42x1.75mm_HandSolder" H 2450 5500 50  0001 C CNN
+F 1 "4.7u" V 2312 5500 50  0000 C CNN
+F 2 "Capacitor_THT:C_Disc_D4.3mm_W1.9mm_P5.00mm" H 2450 5500 50  0001 C CNN
 F 3 "~" H 2450 5500 50  0001 C CNN
 	1    2450 5500
@@
 Text GLabel 1750 6850 0    50   Input ~ 0
 R~W~
-Text Notes 1200 7000 0    50   ~ 0
-Added RW here
 Text Notes 3100 6550 0    50   ~ 0
 Diode + pullup provided by backplane
 Wire Wire Line
 	3150 6350 3100 6350
+$Comp
+L Connector_Generic:Conn_01x14 J2
+U 1 1 61551DA1
+P 6450 3400
+F 0 "J2" H 6530 3392 50  0000 L CNN
+F 1 "Conn_01x14" H 6530 3301 50  0000 L CNN
+F 2 "Connector_PinSocket_2.54mm:PinSocket_1x14_P2.54mm_Vertical" H 6450 3400 50  0001 C CNN
+F 3 "~" H 6450 3400 50  0001 C CNN
+	1    6450 3400
+	1    0    0    -1
+$EndComp
+Wire Wire Line
+	7600 2300 6100 2300
+Wire Wire Line
+	6100 2300 6100 2800
+Wire Wire Line
+	6100 2800 6250 2800
+Text GLabel 6250 2900 0    50   Input ~ 0
+~RAMW~
+Text GLabel 6250 3000 0    50   Input ~ 0
+A13
+Text GLabel 6250 3100 0    50   Input ~ 0
+A8
+Text GLabel 6250 3200 0    50   Input ~ 0
+A9
+Text GLabel 6250 3300 0    50   Input ~ 0
+A11
+$Comp
+L power:GND #PWR0113
+U 1 1 6155B08E
+P 5950 3400
+F 0 "#PWR0113" H 5950 3150 50  0001 C CNN
+F 1 "GND" H 5955 3227 50  0000 C CNN
+F 2 "" H 5950 3400 50  0001 C CNN
+F 3 "" H 5950 3400 50  0001 C CNN
+	1    5950 3400
+	1    0    0    -1
+$EndComp
+Wire Wire Line
+	6250 3400 5950 3400
+Text GLabel 6250 3500 0    50   Input ~ 0
+A10
+Text GLabel 6250 3600 0    50   Input ~ 0
+~RAM_CS~
+Text GLabel 6250 4100 0    50   BiDi ~ 0
+D3
+Text GLabel 6250 4000 0    50   BiDi ~ 0
+D4
+Text GLabel 6250 3900 0    50   BiDi ~ 0
+D5
+Text GLabel 6250 3800 0    50   BiDi ~ 0
+D6
+Text GLabel 6250 3700 0    50   BiDi ~ 0
+D7
 $EndSCHEMATC

Commit message: small updates to this deprecated board
Parts:
- C1, C2, C3, C4: value 4.7u -> 10n
Changed lines of the file:
@@
 P 4800 1700
 F 0 "C3" V 4571 1700 50  0000 C CNN
-F 1 "4.7u" V 4662 1700 50  0000 C CNN
+F 1 "10n" V 4662 1700 50  0000 C CNN
 F 2 "Capacitor_THT:C_Disc_D4.3mm_W1.9mm_P5.00mm" H 4800 1700 50  0001 C CNN
 F 3 "~" H 4800 1700 50  0001 C CNN
@@
 P 7800 2300
 F 0 "C1" V 7571 2300 50  0000 C CNN
-F 1 "4.7u" V 7662 2300 50  0000 C CNN
+F 1 "10n" V 7662 2300 50  0000 C CNN
 F 2 "Capacitor_THT:C_Disc_D4.3mm_W1.9mm_P5.00mm" H 7800 2300 50  0001 C CNN
 F 3 "~" H 7800 2300 50  0001 C CNN
@@
 P 9700 2100
 F 0 "C2" V 9471 2100 50  0000 C CNN
-F 1 "4.7u" V 9562 2100 50  0000 C CNN
+F 1 "10n" V 9562 2100 50  0000 C CNN
 F 2 "Capacitor_THT:C_Disc_D4.3mm_W1.9mm_P5.00mm" H 9700 2100 50  0001 C CNN
 F 3 "~" H 9700 2100 50  0001 C CNN
@@
 P 2450 5500
 F 0 "C4" V 2221 5500 50  0000 C CNN
-F 1 "4.7u" V 2312 5500 50  0000 C CNN
+F 1 "10n" V 2312 5500 50  0000 C CNN
 F 2 "Capacitor_THT:C_Disc_D4.3mm_W1.9mm_P5.00mm" H 2450 5500 50  0001 C CNN
 F 3 "~" H 2450 5500 50  0001 C CNN
