File: Hardware/cpu_backplane/cpu_backplane.sch (KiCad schematic (older format))
At the start: 82 parts, among them J1 USB_B_Micro, J2 Conn_02x02_Odd_Even, J3 Conn_01x06, J4 Conn_01x14, SW1 SW_SPST, U1 74AC161, U4 PAL24, U5 GAL16V8, U6 W65C02SxP, U7 HM62256BLP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

Commit message: DS1813
Parts:
- gave numbers to parts that had none: 2
Changed lines of the file:
@@
 Connection ~ 5350 8250
 $Comp
-L DS1813-10+:DS1813-10+ IC?
+L DS1813-10+:DS1813-10+ IC2
 U 1 1 618021F5
 P 8850 1300
-F 0 "IC?" H 9578 1246 50  0000 L CNN
+F 0 "IC2" H 9578 1246 50  0000 L CNN
 F 1 "DS1813-10+" H 9578 1155 50  0000 L CNN
 F 2 "Package_TO_SOT_THT:TO-92L_Inline" H 9600 1400 50  0001 L CNN
@@
 	8850 1100 9950 1100
 $Comp
-L power:GND #PWR?
+L power:GND #PWR0112
 U 1 1 618B82E0
 P 4800 1350
-F 0 "#PWR?" H 4800 1100 50  0001 C CNN
+F 0 "#PWR0112" H 4800 1100 50  0001 C CNN
 F 1 "GND" H 4805 1177 50  0000 C CNN
 F 2 "" H 4800 1350 50  0001 C CNN
@@
 $EndComp
 $Comp
-L power:+5V #PWR?
+L power:+5V #PWR0136
 U 1 1 618B82E6
 P 4500 1300
-F 0 "#PWR?" H 4500 1150 50  0001 C CNN
+F 0 "#PWR0136" H 4500 1150 50  0001 C CNN
 F 1 "+5V" H 4515 1473 50  0000 C CNN
 F 2 "" H 4500 1300 50  0001 C CNN
@@
 $EndComp
 $Comp
-L DS1813-10+:DS1813-10+ IC?
+L DS1813-10+:DS1813-10+ IC1
 U 1 1 618B82F2
 P 4800 1150
-F 0 "IC?" H 5528 1096 50  0000 L CNN
+F 0 "IC1" H 5528 1096 50  0000 L CNN
 F 1 "DS1813-10+" H 5528 1005 50  0000 L CNN
 F 2 "Package_TO_SOT_THT:TO-92L_Inline" H 5550 1250 50  0001 L CNN
