File: Hardware/cpu_backplane/cpu_backplane.kicad_sch (KiCad schematic)
At the start: 84 parts, among them IC1 DS1813, IC2 DS1813, J1 Barrel_Jack, J2 Conn_02x02_Odd_Even, J3 Conn_01x06, J4 Conn_01x14, Q1 2N3905, SW1 SW_SPST, U1 74AC161, U4 PAL24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

Commit message: update to kicad 6
Parts:
- removed Q1: 2N3905, Package_TO_SOT_THT:TO-92_Inline, symbol Transistor_BJT:2N3905
- added D9: 1N5822, Diode_THT:D_DO-201AD_P15.24mm_Horizontal, symbol Diode:1N5822
- added U2: L7905, Package_TO_SOT_THT:TO-220-3_Vertical, symbol Regulator_Linear:L7905
- SW1: value SW_SPST -> SW
Connections:
- net +5V: now also R7.2, U2.3 (VO); no longer SW1.2 (B)
- net GND: now also U2.1 (GND); no longer R7.2
- net ~{SER_IRQ}: now also R7.1, U9.26 (~{IRQ})
- net at SW1.1 (A): now also D9.1 (K)
- net at J1.1: now also D9.2 (A)
- net ~{SIRQ}: no longer names the net of U5.14 (IO6)
- net ~{SIRQ}: no longer U9.26 (~{IRQ})
- new net: SW1.2 (B), U2.2 (VI)
Other:
- company: (none) -> Six Pixels
- moved on the sheet: C13

Commit message: Add kibot
Parts:
- J1: footprint Connector_BarrelJack:BarrelJack_Horizontal -> w_conn_av:BarrelJack_Horizontal
- SW1: footprint Button_Switch_THT:SW_E-Switch_EG1271_DPDT -> Button_Switch_THT:SW_E-Switch_EG1271_SPDT
Changed lines of the file:
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@@
     (rev "${VERSION}")
     (company "Six Pixels")
+    (comment 1 "Updated power supply to 5.5mm jack")
   )
   (junction (at 101.6 205.74) (diameter 0) (color 0 0 0 0)
@@
     (property "Reference" "SW1" (id 0) (at 48.26 20.701 0))
     (property "Value" "SW" (id 1) (at 48.26 23.0124 0))
-    (property "Footprint" "Button_Switch_THT:SW_E-Switch_EG1271_DPDT" (id 2) (at 48.26 26.67 0)
+    (property "Footprint" "Button_Switch_THT:SW_E-Switch_EG1271_SPDT" (id 2) (at 48.26 26.67 0)
       (effects (font (size 1.27 1.27)) hide)
     )
@@
     (property "Reference" "J1" (id 0) (at 20.32 21.7002 0))
     (property "Value" "Barrel_Jack" (id 1) (at 20.32 24.2371 0))
-    (property "Footprint" "Connector_BarrelJack:BarrelJack_Horizontal" (id 2) (at 21.59 30.226 0)
+    (property "Footprint" "w_conn_av:BarrelJack_Horizontal" (id 2) (at 21.59 30.226 0)
       (effects (font (size 1.27 1.27)) hide)
     )
@@
     )
     (path "/62ec5163-e7ef-4606-8bc5-277e683662d5"
-      (reference "J1") (unit 1) (value "Barrel_Jack") (footprint "Connector_BarrelJack:BarrelJack_Horizontal")
+      (reference "J1") (unit 1) (value "Barrel_Jack") (footprint "w_conn_av:BarrelJack_Horizontal")
     )
     (path "/00000000-0000-0000-0000-000060150e99"
@@
     )
     (path "/00000000-0000-0000-0000-000060031505"
-      (reference "SW1") (unit 1) (value "SW") (footprint "Button_Switch_THT:SW_E-Switch_EG1271_DPDT")
+      (reference "SW1") (unit 1) (value "SW") (footprint "Button_Switch_THT:SW_E-Switch_EG1271_SPDT")
     )
     (path "/00000000-0000-0000-0000-00005ff93a76"
