File: Hardware/proto_board/proto_board.kicad_pcb (KiCad board)
At the start: 2 copper layers, 80.8 x 60.1 mm, 11 parts, among them J1 Conn_01x40, J10 Conn_02x30_Odd_Even, J11 Conn_02x28_Odd_Even, J2 Conn_02x30_Odd_Even, J3 Conn_02x30_Odd_Even, J4 Conn_02x30_Odd_Even, J5 Conn_02x30_Odd_Even, J6 Conn_02x30_Odd_Even, J7 Conn_02x30_Odd_Even, J8 Conn_02x30_Odd_Even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

Commit message: cleanup
Other:
- board text added: "${VERSION}"
Changed lines of the file:
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@@
       (effects (font (size 1 1) (thickness 0.15)))
     )
-    (fp_line (start -1.33 -1.33) (end 0 -1.33) (layer "F.SilkS") (width 0.12))
-    (fp_line (start -1.33 1.27) (end 1.27 1.27) (layer "F.SilkS") (width 0.12))
-    (fp_line (start 1.27 -1.33) (end 3.87 -1.33) (layer "F.SilkS") (width 0.12))
-    (fp_line (start -1.33 1.27) (end -1.33 69.91) (layer "F.SilkS") (width 0.12))
-    (fp_line (start -1.33 0) (end -1.33 -1.33) (layer "F.SilkS") (width 0.12))
-    (fp_line (start 1.27 1.27) (end 1.27 -1.33) (layer "F.SilkS") (width 0.12))
-    (fp_line (start 3.87 -1.33) (end 3.87 69.91) (layer "F.SilkS") (width 0.12))
-    (fp_line (start -1.33 69.91) (end 3.87 69.91) (layer "F.SilkS") (width 0.12))
     (fp_line (start -1.8 -1.8) (end -1.8 70.35) (layer "F.CrtYd") (width 0.05))
     (fp_line (start 4.35 70.35) (end 4.35 -1.8) (layer "F.CrtYd") (width 0.05))
@@
     (effects (font (size 0.8 0.8) (thickness 0.15)))
   )
+  (gr_text "${VERSION}" (at 115.189 129.921) (layer "F.SilkS")
+    (effects (font (size 1.5 1.5) (thickness 0.3)))
+  )
   (gr_text "~{NMI}" (at 122.555 136.525) (layer "F.SilkS")
