File: Hardware/ram_board/ram_board.kicad_sch (KiCad schematic)
At the start: 11 parts, among them J1 Conn_01x40, U1 74HC00, U2 74HC04, U3 IS61C5128AL-10TLI, U5 74HC273

Commit message: Add RAM board + some VGA things
Parts:
- added C7: 100n, Capacitor_THT:C_Disc_D4.3mm_W1.9mm_P5.00mm, symbol Device:C_Small
- added U4: 74HC02, Package_DIP:DIP-14_W7.62mm_Socket, symbol 74xx:74HC02
Connections:
- net +5V: now also C7.2, U4.14 (VCC)
- net CLK: now also U4.3; no longer U1.13
- net GND: now also C7.1, U4.12, U4.7 (GND)
- net ~{CE}: no longer U1.2
- net ~{SLOT_SEL}: now also U4.2; no longer U1.12
- net at U5.11 (Cp): now also U4.1; no longer U1.11
- net at U2.11, U5.19 (Q7): now also U1.2
- new net: U1.12, U1.13, U4.5
- new net: U4.6, U4.8
- new net: U4.11, U4.9
Other:
- note added: "This is wrong"
- moved on the sheet: U1D, U2C

Commit message: fix RAM board ERC and DRC
Connections:
- net GND: now also U1.12, U1.13, U4.11, U4.5, U4.6, U4.8, U4.9
Changed lines of the file:
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@@
   (junction (at 24.13 82.55) (diameter 0) (color 0 0 0 0)
+  )
+  (junction (at 35.56 148.59) (diameter 0) (color 0 0 0 0)
+  )
+  (junction (at 35.56 153.67) (diameter 0) (color 0 0 0 0)
   )
   (junction (at 63.5 83.82) (diameter 0) (color 0 0 0 0)
@@
   )
   (junction (at 148.59 30.48) (diameter 0) (color 0 0 0 0)
+  )
+  (junction (at 35.56 157.48) (diameter 0) (color 0 0 0 0)
   )
   (junction (at 59.69 170.18) (diameter 0) (color 0 0 0 0)
@@
   (junction (at 139.7 36.83) (diameter 0) (color 0 0 0 0)
   )
+  (junction (at 35.56 175.26) (diameter 0) (color 0 0 0 0)
+  )
   (junction (at 133.35 36.83) (diameter 0) (color 0 0 0 0)
   )
   (junction (at 125.73 36.83) (diameter 0) (color 0 0 0 0)
+  )
+  (junction (at 35.56 162.56) (diameter 0) (color 0 0 0 0)
   )
   (junction (at 118.11 31.75) (diameter 0) (color 0 0 0 0)
@@
   )
   (junction (at 241.3 24.13) (diameter 0) (color 0 0 0 0)
+  )
+  (junction (at 35.56 170.18) (diameter 0) (color 0 0 0 0)
   )
   (junction (at 173.99 113.03) (diameter 0) (color 0 0 0 0)
@@
   )
   (wire (pts (xy 106.68 36.83) (xy 113.03 36.83))
+    (stroke (width 0) (type default))
+  )
+  (wire (pts (xy 35.56 170.18) (xy 35.56 175.26))
     (stroke (width 0) (type default))
   )
@@
     (stroke (width 0) (type default))
   )
+  (wire (pts (xy 35.56 157.48) (xy 35.56 162.56))
+    (stroke (width 0) (type default))
+  )
   (wire (pts (xy 224.79 49.53) (xy 241.3 49.53))
     (stroke (width 0) (type default))
@@
     (stroke (width 0) (type default))
   )
+  (wire (pts (xy 35.56 148.59) (xy 35.56 153.67))
+    (stroke (width 0) (type default))
+  )
